File: kicad/simple_ui/simple_ui.kicad_sch (KiCad schematic)
At the start: 59 parts, among them J1 Conn_01x09_Pin, J2 Conn_01x10_Pin, J3 Conn_01x10_Pin, J4 Conn_01x05_Pin, SW1 SW_Push, SW2 SW_Push, SW3 SW_Push, SW4 SW_Push, SW5 SW_Push, SW6 SW_Push, SW7 SW_Push, SW8 SW_Push, SW9 RotaryEncoder_Switch_MP

Commit message: simple ui done
Parts:
- removed J3: Conn_01x10_Pin, Connector_PinSocket_1.27mm:PinSocket_1x10_P1.27mm_Vertical, symbol Connector:Conn_01x10_Pin
- removed RV5, RV6, RV7, RV8: R_Potentiometer, Potentiometer_THT:Potentiometer_Bourns_PTV09A-1_Single_Vertical, symbol Device:R_Potentiometer
- added J3: Conn_01x06_Pin, Connector_PinSocket_1.27mm:PinSocket_1x06_P1.27mm_Vertical, symbol Connector:Conn_01x06_Pin
Connections:
- net GND4: now also J3.6 (Pin_6)
- net POTI1: now also J3.2 (Pin_2)
- net POTI2: now also J3.3 (Pin_3)
- net POTI3: now also J3.4 (Pin_4)
- net POTI4: now also J3.5 (Pin_5)
- net VCC3: now also J3.1 (Pin_1)
Other:
- note added: "7 x Potentiometer PTV09A-4020F-C103"
- note removed: "4 x Potentiometer PTV09A-4020F-C103"
