File: kicad/simple_ui/simple_ui.kicad_pcb (KiCad board)
At the start: 2 copper layers, 59 parts, among them J1 Conn_01x09_Pin, J2 Conn_01x10_Pin, J3 Conn_01x10_Pin, J4 Conn_01x05_Pin, SW1 SW_Push, SW2 SW_Push, SW3 SW_Push, SW4 SW_Push, SW5 SW_Push, SW6 SW_Push, SW7 SW_Push, SW8 SW_Push, SW9 RotaryEncoder_Switch_MP

Commit message: simple ui done
Parts:
- removed RV5, RV6, RV7, RV8: R_Potentiometer, Potentiometer_THT:Potentiometer_Bourns_PTV09A-1_Single_Vertical
- J3: value Conn_01x10_Pin -> Conn_01x06_Pin; footprint Connector_PinSocket_1.27mm:PinSocket_1x10_P1.27mm_Vertical -> Connector_PinSocket_1.27mm:PinSocket_1x06_P1.27mm_Vertical
- moved SW8 185.0 mm to (228.0, 81.0), turned to 180 degrees
- moved C8 177.8 mm to (233.0, 81.0), turned to -90 degrees
- moved SW7 172.5 mm to (216.0, 81.0), turned to 180 degrees
- moved C7 165.7 mm to (221.0, 81.0), turned to -90 degrees
- moved RV4 161.9 mm to (224.5, 100.0), turned to -90 degrees
- moved SW6 160.3 mm to (204.0, 81.0), turned to 180 degrees
- moved R16 154.5 mm to (223.0, 81.0), turned to 90 degrees
- moved C6 153.6 mm to (209.0, 81.0), turned to -90 degrees
- moved C11 148.9 mm to (207.0, 57.0), turned to -90 degrees
- moved SW5 148.3 mm to (192.0, 81.0), turned to 180 degrees
- moved R15 142.5 mm to (211.0, 81.0), turned to 90 degrees
- moved R19 142.5 mm to (207.0, 53.5), turned to -90 degrees
- moved C5 141.5 mm to (197.0, 81.0), turned to -90 degrees
- moved RV3 139.1 mm to (197.0, 100.0), turned to -90 degrees
- moved SW4 136.7 mm to (180.0, 81.0), turned to 180 degrees
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Connections:
- J3 pad 6: /POTI5 -> GND4
Routing:
- net VCC2: track 0.00 -> 160.5 mm
- net VCC3: track 0.00 -> 104.6 mm, vias 0 -> 1
- net GND2: track 0.00 -> 68.6 mm, vias 0 -> 8
- net /BTN8: track 0.00 -> 50.6 mm
- net /BTN1: track 0.00 -> 48.6 mm
- net /POTI1: track 0.00 -> 45.2 mm
- net /POTI4: track 0.00 -> 42.3 mm
- net /BTN7: track 0.00 -> 39.7 mm
- net VCC5: track 0.00 -> 39.6 mm, vias 0 -> 2
- net /BTN2: track 0.00 -> 38.0 mm
- net GND1: track 0.00 -> 37.2 mm, vias 0 -> 7
- net /ROT1_B: track 0.00 -> 30.8 mm
- net /BTN6: track 0.00 -> 29.1 mm
- net /ROT1_A: track 0.00 -> 27.8 mm
- net /BTN3: track 0.00 -> 27.4 mm
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- added copper zone on B.Cu, net GND1
- added copper zone on B.Cu, net GND2
- added copper zone on B.Cu, net GND4
- added copper zone on B.Cu, net GND5
Other:
- board outline added: 100 x 70 mm
- board text added: "simple user interface - LEDs 2024-08-26, MEgli"
- board text added: "simple user interface - buttons 2024-08-26, MEgli"
- board text added: "simple user interface - potentiometer 2024-08-26, MEgli"
- board text added: "simple user interface - rotary en 2024-08-26, MEgli"

Commit message: ready to order pcbs
Other:
- outline, holes or cut-outs redrawn
